Commit message: modified:   description/robot.urdf.xacro 	modified:   description/robot_core.xacro

File: description/robot.urdf.xacro (robot description, xacro)
@@ -1,4 +1,4 @@
 <?xml version="1.0"?>
 <robot xmlns:xacro="http://www.ros.org/wiki/xacro"  name="robot">
- <xacro:inclde filename="robot_core.xacro" />
+<link name="base_link"></link>
 </robot>

Commit message: modified:   description/robot.urdf.xacro 	modified:   description/robot_core.xacro

File: description/robot.urdf.xacro (robot description, xacro)
@@ -1,4 +1,4 @@
 <?xml version="1.0"?>
 <robot xmlns:xacro="http://www.ros.org/wiki/xacro"  name="robot">
-<link name="base_link"></link>
+<xacro:include filename="robot_core.xacro" />
 </robot>

Commit message: new file:   description/lidar.xacro 	modified:   description/robot.urdf.xacro 	modified:   description/robot_core.xacro

File: description/robot.urdf.xacro (robot description, xacro)
@@ -3,3 +3,4 @@
 <xacro:include filename="robot_core.xacro" />
 <xacro:include filename="gazebo_control.xacro" />
+<xacro:include filename="lidar.xaro" />
 </robot>

File: description/robot_core.xacro (robot description, xacro)
@@ -13,4 +13,7 @@
  <material name="black">
         <color rgba="0 0 0 1" />
+    </material>
+     <material name="red">
+        <color rgba="1 0 0 1" />
     </material>
     <!--base link-->
