Commit message: modified:   description/lidar.xacro

File: description/lidar.xacro (robot description, xacro)
@@ -22,33 +22,3 @@
          </xacro:inertial_cylinder>
     </link>
-    <gazebo reference="laser_frame">
-        <material>Gazebo/Red</material>
-        <sensor name="laser" type="ray">
-            <pose>0 0 0 0 0 0</pose>
-            <visualize>true</visualize>
-            <update_rate>10</update_rate>
-            <ray>
-                <scan>
-                    <horizontal>
-                        <samples>360</samples>
-                        <resolution>1</resolution>
-                        <min_angle>-3.14</min_angle>
-                        <max_angle>3.14</max_angle>
-                    </horizontal>
-                </scan>
-                <range>
-                    <min>0.3</min>
-                    <max>12</max>
-                    <resolution>0.01</resolution>
-                </range>
-            </ray>
-            <plugin name="laser_controller" filename="libgazebo_ros_ray_sensor.so">
-                <ros>
-                    <argument>-/out:=scan</argument>
-                </ros>
-                <output_type>sensor_msgs/LaserScan</output_type>
-                <frame_name>laser_frame</frame_name>
-            </plugin>
-        </sensor>
-    </gazebo>
 </robot>

Commit message: modified:   description/lidar.xacro

File: description/lidar.xacro (robot description, xacro)
@@ -1,24 +1,24 @@
 <?xml version="1.0"?>
-<robot xmlns:xacro="http://www.ros.org/wiki/xacro"  >
-   <joint name="laser_joint" type="fixed">
+<robot xmlns:xacro="http://www.ros.org/wiki/xacro">
+<joint name="laser_joint" type="fixed">
     <parent link="chassis"/>
     <child link="laser_frame"/>
     <origin xyz="0.1 0 0.175" rpy="0 0 0"/>
-    </joint>
-    <link name="laser_frame">
-        <visual>
-             <geometry>
-                  <cylinder radius="0.05" length="0.04"/>
-             </geometry>
-             <material name="red"/>
-         </visual>
-         <collision>
-             <geometry>
-                <cylinder radius="0.05" length="0.04"/>
-              </geometry>
-         </collision>
-         <xacro:inertial_cylinder mass="0.1" length="0.04" radius="0.05">
-             <origin xyz="0 0 0" rpy="0 0 0"/>
-         </xacro:inertial_cylinder>
-    </link>
+</joint>
+<link name="laser_frame">
+     <visual>
+        <geometry>
+            <cylinder radius="0.05" length="0.04"/>
+        </geometry>
+        <material name="red"/>
+    </visual>
+     <collision>
+        <geometry>
+            <cylinder radius="0.05" length="0.04"/>
+        </geometry>
+    </collision>
+    <xacro:inertial_cylinder mass="0.1" length="0.04" radius="0.05">
+        <origin xyz="0 0 0" rpy="0 0 0"/>
+    </xacro:inertial_cylinder>
+</link>
 </robot>

Commit message: modified:   description/lidar.xacro

File: description/lidar.xacro (robot description, xacro)
@@ -7,5 +7,5 @@
 </joint>
 <link name="laser_frame">
-     <visual>
+    <visual>
         <geometry>
             <cylinder radius="0.05" length="0.04"/>
@@ -13,8 +13,8 @@
         <material name="red"/>
     </visual>
-     <collision>
+    <collision>
         <geometry>
             <cylinder radius="0.05" length="0.04"/>
-        </geometry>
+        <geometry>
     </collision>
     <xacro:inertial_cylinder mass="0.1" length="0.04" radius="0.05">

Commit message: modified:   description/lidar.xacro

File: description/lidar.xacro (robot description, xacro)
@@ -11,5 +11,5 @@
             <cylinder radius="0.05" length="0.04"/>
         </geometry>
-        <material name="red"/>
+        <material name="Red"/>
     </visual>
     <collision>

Commit message: modified:   description/lidar.xacro

File: description/lidar.xacro (robot description, xacro)
@@ -1,24 +1,24 @@
 <?xml version="1.0"?>
 <robot xmlns:xacro="http://www.ros.org/wiki/xacro">
-<joint name="laser_joint" type="fixed">
-    <parent link="chassis"/>
-    <child link="laser_frame"/>
-    <origin xyz="0.1 0 0.175" rpy="0 0 0"/>
-</joint>
-<link name="laser_frame">
-    <visual>
-        <geometry>
-            <cylinder radius="0.05" length="0.04"/>
-        </geometry>
-        <material name="Red"/>
-    </visual>
-    <collision>
-        <geometry>
-            <cylinder radius="0.05" length="0.04"/>
-        <geometry>
-    </collision>
-    <xacro:inertial_cylinder mass="0.1" length="0.04" radius="0.05">
-        <origin xyz="0 0 0" rpy="0 0 0"/>
-    </xacro:inertial_cylinder>
-</link>
+    <joint name="laser_joint" type="fixed">
+        <parent link="chassis"/>
+        <child link="laser_frame"/>
+        <origin xyz="0.1 0 0.175" rpy="0 0 0"/>
+    </joint>
+    <link name="laser_frame">
+        <visual>
+            <geometry>
+                <cylinder radius="0.05" length="0.04"/>
+            </geometry>
+            <material name="red"/>
+        </visual>
+        <collision>
+            <geometry>
+                <cylinder radius="0.05" length="0.04"/>
+            <geometry>
+        </collision>
+        <xacro:inertial_cylinder mass="0.1" length="0.04" radius="0.05">
+            <origin xyz="0 0 0" rpy="0 0 0"/>
+        </xacro:inertial_cylinder>
+    </link>
 </robot>
