Commit message: modified:   description/robot_core.xacro

File: description/robot_core.xacro (robot description, xacro)
@@ -19,17 +19,3 @@
     <link name="base_link">
     </link>
-    <joint name="chassis_joint" type="fixed">
-        <parent link="base_link"/>
-        <child link="chassis"/>
-        <origin xyz="-0.1 0 0"/>
-    </joint>
-      <link name="chassis">
-        <visual>
-            <origin xyz="0.15 0 0.075"/>
-            <geometry>
-                <box size="0.3 0.3 0.15"/>
-            </geometry>
-            <material name="white"/>
-        </visual>
-      </link>
 </robot>

Commit message: modified:   description/robot_core.xacro

File: description/robot_core.xacro (robot description, xacro)
@@ -13,8 +13,4 @@
         <color rgba="0 0 0 1" />
     </material>
-    <material name="red">
-        <color rgba="1 0 0 1" />
-    </material>
-    <!-- BASE LINK-->
     <link name="base_link">
     </link>

Commit message: modified:   description/robot_core.xacro

File: description/robot_core.xacro (robot description, xacro)
@@ -26,5 +26,5 @@
                 <box size="0.3 0.3 0.15"/>
             </geometry>
-            <material name="white"/>
+            <material name="White"/>
         </visual>
 </robot>

Commit message: modified:   description/robot_core.xacro

File: description/robot_core.xacro (robot description, xacro)
@@ -15,16 +15,17 @@
 <link name="base_link">
 </link>
- <joint name="chassis_joint" type="fixed">
-        <parent link="base_link"/>
-        <child link="chassis"/>
-        <origin xyz="-0.1 0 0"/>
-    </joint>
-    <link name="chassis">
-        <visual>
-            <origin xyz="0.15 0 0.075"/>
-            <geometry>
-                <box size="0.3 0.3 0.15"/>
-            </geometry>
-            <material name="White"/>
-        </visual>
+<joint name="chassi_joint" type="fixed">
+    <parent link="base_link"/>
+    <child link="chassis"/>
+    <origin xyz="-0.1 0 0"/>
+</joint>
+<link name="chassis">
+    <visual>
+        <origin xyz="0.15 0 0.075"/>
+        <geometry>
+            <box size="0.3 0.3 0.15"/>
+        </geometry>
+        <material name="white"/>
+    </visual>
+</link>
 </robot>

Commit message: modified:   description/robot_core.xacro

File: description/robot_core.xacro (robot description, xacro)
@@ -31,3 +31,33 @@
     </visual>
 </link>
+    <!--left wheel link-->
+<joint name="left_wheel_joint" type="continuous">
+    <parent link="base_link"/>
+    <child link="left_wheel"/>
+    <origin xyz="0 0.175 0" rpy="-${pi/2} 0 0"/>
+    <axis xyz="0 0 1"/>
+</joint>
+<link name="left_wheel">
+    <visual>
+        <geometry>
+            <cylinder radius="0.05" length="0.04"/>
+        </geometry>
+        <material name="blue"/>
+    </visual>
+</link>
+    <!--right wheel link-->
+<joint name="right_wheel_joint" type="continuous">
+    <parent link="base_link"/>
+    <child link="right_wheel"/>
+    <origin xyz="0 -0.175 0" rpy="${pi/2} 0 0"/>
+    <axis xyz="0 0 -1"/>
+</joint>
+<link name="right_wheel">
+    <visual>
+        <geometry>
+            <cylinder radius="0.05" length="0.04"/>
+        </geometry>
+        <material name="blue"/>
+    </visual>
+</link>
 </robot>

Commit message: modified:   description/robot_core.xacro

File: description/robot_core.xacro (robot description, xacro)
@@ -61,3 +61,17 @@
     </visual>
 </link>
+    <!--caster wheel link-->
+<joint name="caster_wheel_joint" type="fixed">
+    <parent link="chassis"/>
+    <child link="caster_wheel"/>
+    <origin xyz="0.24 0 0"/>
+</joint>
+<link name="caster_wheel">
+    <visual>
+        <geometry>
+            <sphere radius="0.05"/>
+        </geometry>
+        <material name="black"/>
+    </visual>
+</link>
 </robot>

Commit message: modified:   description/robot_core.xacro

File: description/robot_core.xacro (robot description, xacro)
@@ -30,4 +30,10 @@
         <material name="white"/>
     </visual>
+    <collision>
+        <origin xyz="0.15 0 0.075"/>
+        <geometry>
+            <box size="0.3 0.3 0.15"/>
+        </geometry>
+    </collision>
 </link>
     <!--left wheel link-->
@@ -45,4 +51,9 @@
         <material name="blue"/>
     </visual>
+     <collision>
+        <geometry>
+            <cylinder radius="0.05" length="0.04"/>
+        </geometry>
+    </collision>
 </link>
     <!--right wheel link-->
@@ -60,4 +71,9 @@
         <material name="blue"/>
     </visual>
+    <collision>
+        <geometry>
+            <cylinder radius="0.05" length="0.04"/>
+        </geometry>
+    </collision>
 </link>
     <!--caster wheel link-->
@@ -74,4 +90,9 @@
         <material name="black"/>
     </visual>
+    <collision>
+        <geometry>
+            <sphere radius="0.05"/>
+        </geometry>
+    </collision>
 </link>
 </robot>

Commit message: new file:   description/inertial_macros.xacro 	modified:   description/robot_core.xacro

File: description/robot_core.xacro (robot description, xacro)
@@ -1,4 +1,5 @@
 <?xml version="1.0"?>
 <robot xmlns:xacro="http://www.ros.org/wiki/xacro"  >
+<xacro:include filename="inertial_macros.xacro" />
  <material name="white">
         <color rgba="1 1 1 1" />
@@ -36,4 +37,7 @@
         </geometry>
     </collision>
+    <xacro:inertial_box mass="0.5" x="0.3" y="0.3" z="0.15">
+        <origin xyz="0.15 0 0.075" rpy="0 0 0"/>
+    </xacro:inertial_box>
 </link>
     <!--left wheel link-->
@@ -56,4 +60,7 @@
         </geometry>
     </collision>
+    <xacro:inertial_cylinder mass="0.1" length="0.04" radius="0.05">
+        <origin xyz="0 0 0" rpy="0 0 0"/>
+    </xacro:inertial_cylinder>
 </link>
     <!--right wheel link-->
@@ -76,4 +83,7 @@
         </geometry>
     </collision>
+      <xacro:inertial_cylinder mass="0.1" length="0.04" radius="0.05">
+        <origin xyz="0 0 0" rpy="0 0 0"/>
+    </xacro:inertial_cylinder>
 </link>
     <!--caster wheel link-->
@@ -95,4 +105,7 @@
         </geometry>
     </collision>
+    <xacro:inertial_sphere mass="0.1" radius="0.05">
+        <origin xyz="0 0 0" rpy="0 0 0"/>
+    </xacro:inertial_sphere>
 </link>
 </robot>

Commit message: modified:   description/robot_core.xacro

File: description/robot_core.xacro (robot description, xacro)
@@ -41,4 +41,7 @@
     </xacro:inertial_box>
 </link>
+<gazebo reference="chassis">
+    <material>Gazebo/White</material>
+</gazebo>
     <!--left wheel link-->
 <joint name="left_wheel_joint" type="continuous">
@@ -64,4 +67,7 @@
     </xacro:inertial_cylinder>
 </link>
+<gazebo reference="left_wheel">
+    <material>Gazebo/Blue</material>
+</gazebo>
     <!--right wheel link-->
 <joint name="right_wheel_joint" type="continuous">
@@ -87,4 +93,7 @@
     </xacro:inertial_cylinder>
 </link>
+<gazebo reference="right_wheel">
+    <material>Gazebo/Blue</material>
+</gazebo>
     <!--caster wheel link-->
 <joint name="caster_wheel_joint" type="fixed">
@@ -109,3 +118,6 @@
     </xacro:inertial_sphere>
 </link>
+<gazebo reference="caster_wheel">
+    <material>Gazebo/Black</material>
+</gazebo>
 </robot>

Commit message: modified:   description/robot_core.xacro

File: description/robot_core.xacro (robot description, xacro)
@@ -20,4 +20,12 @@
 <link name="base_link">
 </link>
+    <!--base footprint-->
+    <joint name="base_footprint_joint" type="fixed">
+        <parent link="base_link"/>
+        <child link="base_footprint"/>
+        <origin xyz="0 0 0" rpy="0 0 0"/>
+    </joint>
+    <link name="base_footprint">
+    </link>
     <!--chassis link-->
 <joint name="chassi_joint" type="fixed">
